File: bc660_breakoutboard/bc660_breakoutboard.kicad_pcb (KiCad board)
At the start: 2 copper layers, 59.7 x 48.5 mm, 26 parts, among them J1 SMA_CONNECTOR, J2 Conn_01x01_Pin, J3 Conn_01x02_Pin, J4 SIM8051-6-0-14-01-X-REVD, J5 Conn_01x02_Pin, J6 Conn_01x06_Pin, U1 BC660K-GL, U2 ESDS304DBVR

Commit message: Pcb Update
Parts:
- removed U2: ESDS304DBVR, ESDS304DBVR:SOT95P280X145-5N
Routing:
- net Net-(U1-USIM_RST): track 89.9 -> 30.8 mm, vias 0 -> 2
- net Net-(J4-VCC): track 70.8 -> 63.9 mm
- net Net-(U1-USIM_CLK): track 19.2 -> 12.5 mm
- net Net-(U1-USIM_DATA): track 38.5 -> 34.9 mm
Changed lines of the file:
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@@
     )
   )
-  (footprint "ESDS304DBVR:SOT95P280X145-5N" (layer "F.Cu")
-    (at 91.44 88.138 180)
-    (property "Check_prices" "https://www.snapeda.com/parts/ESDS304DBVR/Texas+Instruments/view-part/?ref=eda")
-    (property "Description" "\nQuad 2.3-pF, 3.6-V, ±30-kV ESD protection diode with 12-A 8/20-uS surge rating for USB and Ethernet\n")
-    (property "DigiKey_Part_Number" "")
-    (property "MF" "Texas Instruments")
-    (property "MP" "ESDS304DBVR")
-    (property "Package" "SOT-23-5 Texas Instruments")
-    (property "Purchase-URL" "https://www.snapeda.com/api/url_track_click_mouser/?unipart_id=3215782&manufacturer=Texas Instruments&part_name=ESDS304DBVR&search_term=esds304dbvr")
-    (property "Sheetfile" "bc660_breakoutboard.kicad_sch")
-    (property "Sheetname" "")
-    (property "SnapEDA_Link" "https://www.snapeda.com/parts/ESDS304DBVR/Texas+Instruments/view-part/?ref=snap")
-    (attr smd)
-    (fp_text reference "U2" (at -0.06 -2.508) (layer "F.SilkS")
-        (effects (font (size 0.8 0.8) (thickness 0.15)))
-    )
-    (fp_text value "ESDS304DBVR" (at 5.528 2.508) (layer "F.Fab")
-        (effects (font (size 0.8 0.8) (thickness 0.15)))
-    )
-    (fp_line (start -0.33 -1.45) (end 0.33 -1.45)
-      (stroke (width 0.127) (type solid)) (layer "F.SilkS"))
-    (fp_line (start 0.33 1.45) (end -0.33 1.45)
-      (stroke (width 0.127) (type solid)) (layer "F.SilkS"))
-    (fp_line (start 0.8 -0.335) (end 0.8 0.335)
-      (stroke (width 0.127) (type solid)) (layer "F.SilkS"))
-    (fp_circle (center -2.41 -1.05) (end -2.31 -1.05)
-      (stroke (width 0.2) (type solid)) (fill none) (layer "F.SilkS"))
-    (fp_line (start -2.11 -1.7) (end 2.11 -1.7)
-      (stroke (width 0.05) (type solid)) (layer "F.CrtYd"))
-    (fp_line (start -2.11 1.7) (end -2.11 -1.7)
-      (stroke (width 0.05) (type solid)) (layer "F.CrtYd"))
-    (fp_line (start 2.11 -1.7) (end 2.11 1.7)
-      (stroke (width 0.05) (type solid)) (layer "F.CrtYd"))
-    (fp_line (start 2.11 1.7) (end -2.11 1.7)
-      (stroke (width 0.05) (type solid)) (layer "F.CrtYd"))
-    (fp_line (start -0.8 -1.45) (end 0.8 -1.45)
-      (stroke (width 0.127) (type solid)) (layer "F.Fab"))
-    (fp_line (start -0.8 1.45) (end -0.8 -1.45)
-      (stroke (width 0.127) (type solid)) (layer "F.Fab"))
-    (fp_line (start 0.8 -1.45) (end 0.8 1.45)
-      (stroke (width 0.127) (type solid)) (layer "F.Fab"))
-    (fp_line (start 0.8 1.45) (end -0.8 1.45)
-      (stroke (width 0.127) (type solid)) (layer "F.Fab"))
-    (fp_circle (center -2.41 -1.05) (end -2.31 -1.05)
-      (stroke (width 0.2) (type solid)) (fill none) (layer "F.Fab"))
-    (pad "1" smd roundrect (at -1.255 -0.95 180) (size 1.21 0.59) (layers "F.Cu" "F.Paste" "F.Mask") (roundrect_rratio 0.15)
-      (net 2 "Net-(J4-VCC)") (pinfunction "I/O1") (pintype "bidirectional") (solder_mask_margin 0.102))
-    (pad "2" smd roundrect (at -1.255 0 180) (size 1.21 0.59) (layers "F.Cu" "F.Paste" "F.Mask") (roundrect_rratio 0.15)
-      (net 4 "GND") (pinfunction "GND") (pintype "power_in") (solder_mask_margin 0.102))
-    (pad "3" smd roundrect (at -1.255 0.95 180) (size 1.21 0.59) (layers "F.Cu" "F.Paste" "F.Mask") (roundrect_rratio 0.15)
-      (net 6 "Net-(U1-USIM_CLK)") (pinfunction "I/O2") (pintype "bidirectional") (solder_mask_margin 0.102))
-    (pad "4" smd roundrect (at 1.255 0.95 180) (size 1.21 0.59) (layers "F.Cu" "F.Paste" "F.Mask") (roundrect_rratio 0.15)
-      (net 5 "Net-(U1-USIM_RST)") (pinfunction "I/O3") (pintype "bidirectional") (solder_mask_margin 0.102))
-    (pad "5" smd roundrect (at 1.255 -0.95 180) (size 1.21 0.59) (layers "F.Cu" "F.Paste" "F.Mask") (roundrect_rratio 0.15)
-      (net 3 "Net-(U1-USIM_DATA)") (pinfunction "I/O4") (pintype "bidirectional") (solder_mask_margin 0.102))
-  )
   (footprint "Resistor_SMD:R_0805_2012Metric_Pad1.20x1.40mm_HandSolder" (layer "F.Cu")
     (at 113.03 67.072 -90)
@@
   (segment (start 88.334 94.292) (end 88.392 94.234) (width 0.254) (layer "F.Cu") (net 2))
   (segment (start 88.646 93.98) (end 88.392 94.234) (width 0.254) (layer "F.Cu") (net 2))
-  (segment (start 92.695 89.931) (end 88.392 94.234) (width 0.254) (layer "F.Cu") (net 2))
   (segment (start 73.239 88.559) (end 73.152 88.472) (width 0.254) (layer "F.Cu") (net 2))
   (segment (start 83.566 94.292) (end 79.493 90.219) (width 0.254) (layer "F.Cu") (net 2))
   (segment (start 74.899 90.219) (end 73.239 88.559) (width 0.254) (layer "F.Cu") (net 2))
   (segment (start 101.482 93.98) (end 88.646 93.98) (width 0.254) (layer "F.Cu") (net 2))
-  (segment (start 92.695 89.088) (end 92.695 89.931) (width 0.254) (layer "F.Cu") (net 2))
   (segment (start 79.493 90.219) (end 74.899 90.219) (width 0.254) (layer "F.Cu") (net 2))
   (segment (start 104.694 90.768) (end 101.482 93.98) (width 0.254) (layer "F.Cu") (net 2))
@@
   (segment (start 100.686577 86.568) (end 101.444 86.568) (width 0.254) (layer "F.Cu") (net 3))
   (segment (start 80.524 86.112) (end 90.424 86.112) (width 0.254) (layer "F.Cu") (net 3))
-  (segment (start 89.253 86.769) (end 89.253 88.156) (width 0.254) (layer "F.Cu") (net 3))
   (segment (start 77.459 83.047) (end 80.524 86.112) (width 0.254) (layer "F.Cu") (net 3))
   (segment (start 90.17 86.112) (end 100.230577 86.112) (width 0.254) (layer "F.Cu") (net 3))
@@
   (segment (start 90.424 86.112) (end 90.17 86.112) (width 0.254) (layer "F.Cu") (net 3))
   (segment (start 78.486 78.486) (end 77.459 79.513) (width 0.254) (layer "F.Cu") (net 3))
-  (segment (start 89.253 88.156) (end 90.185 89.088) (width 0.254) (layer "F.Cu") (net 3))
   (segment (start 76.411 80.561) (end 78.486 78.486) (width 0.254) (layer "F.Cu") (net 3))
-  (segment (start 89.91 86.112) (end 89.253 86.769) (width 0.254) (layer "F.Cu") (net 3))
   (segment (start 98.044 65.997) (end 101.054 65.997) (width 0.254) (layer "F.Cu") (net 4))
   (segment (start 75.692 78.486) (end 75.946 78.486) (width 0.254) (layer "F.Cu") (net 4))
-  (segment (start 83.8415 106.934) (end 81.026 104.1185) (width 0.254) (layer "F.Cu") (net 5))
-  (segment (start 113.786577 87.668) (end 121.158 95.039423) (width 0.254) (layer "F.Cu") (net 5))
-  (segment (start 121.158 106.934) (end 83.8415 106.934) (width 0.254) (layer "F.Cu") (net 5))
-  (segment (start 101.444 87.668) (end 113.786577 87.668) (width 0.254) (layer "F.Cu") (net 5))
+  (segment (start 101.444 87.668) (end 93.726 87.668) (width 0.254) (layer "F.Cu") (net 5))
+  (segment (start 93.726 87.668) (end 93.256 87.668) (width 0.254) (layer "F.Cu") (net 5))
   (segment (start 81.026 102.108) (end 81.026 104.1185) (width 0.254) (layer "F.Cu") (net 5))
-  (segment (start 100.686577 87.668) (end 101.444 87.668) (width 0.254) (layer "F.Cu") (net 5))
-  (segment (start 121.158 95.039423) (end 121.158 106.934) (width 0.254) (layer "F.Cu") (net 5))
-  (segment (start 90.185 87.188) (end 90.807 86.566) (width 0.254) (layer "F.Cu") (net 5))
-  (segment (start 90.807 86.566) (end 99.584577 86.566) (width 0.254) (layer "F.Cu") (net 5))
-  (segment (start 99.584577 86.566) (end 100.686577 87.668) (width 0.254) (layer "F.Cu") (net 5))
-  (segment (start 92.695 87.188) (end 94.742 87.188) (width 0.254) (layer "F.Cu") (net 6))
-  (segment (start 94.742 87.188) (end 98.964 87.188) (width 0.254) (layer "F.Cu") (net 6))
-  (segment (start 94.742 92.4345) (end 94.742 89.916) (width 0.254) (layer "F.Cu") (net 6))
-  (segment (start 92.964 92.964) (end 94.742 91.186) (width 0.254) (layer "F.Cu") (net 6))
-  (segment (start 94.742 89.916) (end 94.742 87.188) (width 0.254) (layer "F.Cu") (net 6))
-  (segment (start 98.964 87.188) (end 100.544 88.768) (width 0.254) (layer "F.Cu") (net 6))
-  (segment (start 100.544 88.768) (end 101.444 88.768) (width 0.254) (layer "F.Cu") (net 6))
-  (segment (start 94.742 91.186) (end 94.742 89.916) (width 0.254) (layer "F.Cu") (net 6))
-  (segment (start 95.25 92.9425) (end 94.742 92.4345) (width 0.254) (layer "F.Cu") (net 6))
+  (segment (start 93.256 87.668) (end 93.218 87.63) (width 0.254) (layer "F.Cu") (net 5))
+  (via (at 93.218 87.63) (size 0.8) (drill 0.4) (layers "F.Cu" "B.Cu") (net 5))
+  (via (at 81.026 103.124) (size 0.8) (drill 0.4) (layers "F.Cu" "B.Cu") (net 5))
+  (segment (start 93.218 90.932) (end 81.026 103.124) (width 0.254) (layer "B.Cu") (net 5))
+  (segment (start 93.218 87.63) (end 93.218 90.932) (width 0.254) (layer "B.Cu") (net 5))
+  (segment (start 95.25 92.9425) (end 92.9855 92.9425) (width 0.25) (layer "F.Cu") (net 6))
+  (segment (start 92.964 92.964) (end 97.16 88.768) (width 0.254) (layer "F.Cu") (net 6))
+  (segment (start 92.9855 92.9425) (end 92.964 92.964) (width 0.25) (layer "F.Cu") (net 6))
+  (segment (start 97.16 88.768) (end 101.444 88.768) (width 0.254) (layer "F.Cu") (net 6))
   (segment (start 100.686577 82.168) (end 101.444 82.168) (width 0.254) (layer "F.Cu") (net 7))
   (segment (start 92.202 73.683423) (end 100.686577 82.168) (width 0.254) (layer "F.Cu") (net 7))
