File: bc660_breakoutboard/bc660_breakoutboard.kicad_sch (KiCad schematic)
At the start: 23 parts, among them J2 Conn_01x12_Pin, J3 Conn_Coaxial, J4 SIM8051-6-0-14-01-X-REVD, U1 BC660K-GL, U2 ESDS304DBVR

Commit message: update pcb design
Parts:
- removed J2: Conn_01x12_Pin, Connector_PinHeader_2.54mm:PinHeader_1x12_P2.54mm_Vertical, symbol Connector:Conn_01x12_Pin
- removed J3: Conn_Coaxial, symbol Connector:Conn_Coaxial
- added J1: SMA_CONNECTOR, SMA_CONNECTOR:LPRS_SMA_CONNECTOR, symbol SMA_CONNECTOR:SMA_CONNECTOR
- added J2: Conn_01x01_Pin, Connector_PinHeader_2.54mm:PinHeader_1x01_P2.54mm_Vertical, symbol Connector:Conn_01x01_Pin
- added J3, J5: Conn_01x02_Pin, Connector_PinHeader_2.54mm:PinHeader_1x02_P2.54mm_Vertical, symbol Connector:Conn_01x02_Pin
- added J6: Conn_01x06_Pin, Connector_PinHeader_2.54mm:PinHeader_1x06_P2.54mm_Vertical, symbol Connector:Conn_01x06_Pin
Connections:
- net GND: now also J1.G1, J1.G2, J1.G3, J1.G4, J3.1 (Pin_1); no longer U1.16 (NETLIGHT)
- net at R7.1: now also J5.1 (Pin_1)
- net at C6.2, C7.2, C8.2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: now also J3.2 (Pin_2)
- net at R5.1: now also J6.4 (Pin_4)
- net at R6.1: now also J6.3 (Pin_3)
- net at R8.1: now also J5.2 (Pin_2)
- net at R9.2: now also J6.6 (Pin_6)
- net at U1.7 (~{BOOT}): now also J2.1 (Pin_1)
- net at U1.15 (~{RESET}): now also J6.1 (Pin_1)
- net at U1.19 (PSM_EINT): now also J6.5 (Pin_5)
- net at U1.35 (ANT_RF): now also J1.1
- new net: J6.2 (Pin_2), U1.16 (NETLIGHT)
- no-connect marks 8 -> 9

Commit message: Pcb Update
Parts:
- removed U2: ESDS304DBVR, ESDS304DBVR:SOT95P280X145-5N, symbol ESDS304DBVR:ESDS304DBVR
Changed lines of the file:
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@@
   (junction (at 130.81 54.61) (diameter 0) (color 0 0 0 0)
   )
-  (junction (at 165.1 64.77) (diameter 0) (color 0 0 0 0)
-  )
   (junction (at 113.03 45.72) (diameter 0) (color 0 0 0 0)
   )
@@
   (junction (at 154.94 62.23) (diameter 0) (color 0 0 0 0)
   )
-  (junction (at 167.64 67.31) (diameter 0) (color 0 0 0 0)
-  )
   (junction (at 172.72 67.31) (diameter 0) (color 0 0 0 0)
   )
@@
   )
   (junction (at 201.93 62.23) (diameter 0) (color 0 0 0 0)
-  )
-  (junction (at 162.56 62.23) (diameter 0) (color 0 0 0 0)
-  )
-  (junction (at 170.18 69.85) (diameter 0) (color 0 0 0 0)
   )
   (no_connect (at 85.09 82.55))
@@
   (no_connect (at 130.81 80.01))
   (no_connect (at 130.81 57.15))
-  (bus_entry (at 162.56 46.99) (size 2.54 2.54)
-    (stroke (width 0) (type default))
-  )
   (wire (pts (xy 67.31 97.79) (xy 76.2 97.79))
     (stroke (width 0) (type default))
@@
     (stroke (width 0) (type default))
   )
-  (wire (pts (xy 162.56 53.34) (xy 162.56 62.23))
-    (stroke (width 0) (type default))
-  )
   (wire (pts (xy 251.46 68.58) (xy 251.46 82.55))
     (stroke (width 0) (type default))
@@
     (stroke (width 0) (type default))
   )
-  (wire (pts (xy 165.1 64.77) (xy 190.5 64.77))
+  (wire (pts (xy 163.83 64.77) (xy 190.5 64.77))
     (stroke (width 0) (type default))
   )
@@
     (stroke (width 0) (type default))
   )
-  (wire (pts (xy 170.18 53.34) (xy 170.18 69.85))
-    (stroke (width 0) (type default))
-  )
-  (wire (pts (xy 130.81 67.31) (xy 167.64 67.31))
+  (wire (pts (xy 130.81 67.31) (xy 172.72 67.31))
     (stroke (width 0) (type default))
   )
@@
     (stroke (width 0) (type default))
   )
-  (wire (pts (xy 167.64 53.34) (xy 167.64 67.31))
-    (stroke (width 0) (type default))
-  )
   (wire (pts (xy 224.79 64.77) (xy 224.79 66.04))
     (stroke (width 0) (type default))
@@
     (stroke (width 0) (type default))
   )
-  (wire (pts (xy 170.18 69.85) (xy 181.61 69.85))
+  (wire (pts (xy 130.81 69.85) (xy 181.61 69.85))
     (stroke (width 0) (type default))
   )
@@
     (stroke (width 0) (type default))
   )
-  (wire (pts (xy 163.83 64.77) (xy 165.1 64.77))
-    (stroke (width 0) (type default))
-  )
   (wire (pts (xy 83.82 97.79) (xy 85.09 97.79))
     (stroke (width 0) (type default))
@@
     (stroke (width 0) (type default))
   )
-  (wire (pts (xy 167.64 67.31) (xy 172.72 67.31))
-    (stroke (width 0) (type default))
-  )
   (wire (pts (xy 71.12 82.55) (xy 71.12 87.63))
     (stroke (width 0) (type default))
   )
-  (wire (pts (xy 130.81 69.85) (xy 170.18 69.85))
-    (stroke (width 0) (type default))
-  )
   (wire (pts (xy 163.83 64.77) (xy 163.83 74.93))
     (stroke (width 0) (type default))
@@
     (stroke (width 0) (type default))
   )
-  (wire (pts (xy 165.1 53.34) (xy 165.1 64.77))
-    (stroke (width 0) (type default))
-  )
   (wire (pts (xy 172.72 67.31) (xy 190.5 67.31))
     (stroke (width 0) (type default))
@@
     (stroke (width 0) (type default))
   )
-  (wire (pts (xy 162.56 62.23) (xy 201.93 62.23))
-    (stroke (width 0) (type default))
-  )
   (wire (pts (xy 130.81 64.77) (xy 163.83 64.77))
     (stroke (width 0) (type default))
@@
     (stroke (width 0) (type default))
   )
-  (wire (pts (xy 154.94 62.23) (xy 162.56 62.23))
+  (wire (pts (xy 154.94 62.23) (xy 201.93 62.23))
     (stroke (width 0) (type default))
   )
@@
         (path "/d627ecd8-d3ea-468a-86f8-a115d49eee0e"
           (reference "J2") (unit 1)
-        )
-      )
-    )
-  )
-  (symbol (lib_id "ESDS304DBVR:ESDS304DBVR") (at 170.18 35.56 90) (unit 1)
-    (in_bom yes) (on_board yes) (dnp no) (fields_autoplaced)
-    (property "Reference" "U2" (at 181.61 34.925 90)
-      (effects (font (size 1.27 1.27)) (justify right))
-    )
-    (property "Value" "ESDS304DBVR" (at 181.61 37.465 90)
-      (effects (font (size 1.27 1.27)) (justify right))
-    )
-    (property "Footprint" "ESDS304DBVR:SOT95P280X145-5N" (at 170.18 35.56 0)
-      (effects (font (size 1.27 1.27)) (justify bottom) hide)
-    )
-    (property "Datasheet" "" (at 170.18 35.56 0)
-      (effects (font (size 1.27 1.27)) hide)
-    )
-    (property "DigiKey_Part_Number" "" (at 170.18 35.56 0)
-      (effects (font (size 1.27 1.27)) (justify bottom) hide)
-    )
-    (property "MF" "Texas Instruments" (at 170.18 35.56 0)
-      (effects (font (size 1.27 1.27)) (justify bottom) hide)
-    )
-    (property "Purchase-URL" "https://www.snapeda.com/api/url_track_click_mouser/?unipart_id=3215782&manufacturer=Texas Instruments&part_name=ESDS304DBVR&search_term=esds304dbvr" (at 170.18 35.56 0)
-      (effects (font (size 1.27 1.27)) (justify bottom) hide)
-    )
-    (property "Package" "SOT-23-5 Texas Instruments" (at 170.18 35.56 0)
-      (effects (font (size 1.27 1.27)) (justify bottom) hide)
-    )
-    (property "SnapEDA_Link" "https://www.snapeda.com/parts/ESDS304DBVR/Texas+Instruments/view-part/?ref=snap" (at 170.18 35.56 0)
-      (effects (font (size 1.27 1.27)) (justify bottom) hide)
-    )
-    (property "MP" "ESDS304DBVR" (at 170.18 35.56 0)
-      (effects (font (size 1.27 1.27)) (justify bottom) hide)
-    )
-    (property "Description" "\nQuad 2.3-pF, 3.6-V, ±30-kV ESD protection diode with 12-A 8/20-uS surge rating for USB and Ethernet\n" (at 170.18 35.56 0)
-      (effects (font (size 1.27 1.27)) (justify bottom) hide)
-    )
-    (property "Check_prices" "https://www.snapeda.com/parts/ESDS304DBVR/Texas+Instruments/view-part/?ref=eda" (at 170.18 35.56 0)
-      (effects (font (size 1.27 1.27)) (justify bottom) hide)
-    )
-    (pin "1")
-    (pin "2")
-    (pin "3")
-    (pin "4")
-    (pin "5")
-    (instances
-      (project "bc660_breakoutboard"
-        (path "/d627ecd8-d3ea-468a-86f8-a115d49eee0e"
-          (reference "U2") (unit 1)
         )
       )
@@
         )
       )
-    )
-  )
-  (symbol (lib_id "power:GND") (at 162.56 17.78 180) (unit 1)
-    (in_bom yes) (on_board yes) (dnp no) (fields_autoplaced)
-    (property "Reference" "#PWR05" (at 162.56 11.43 0)
-      (effects (font (size 1.27 1.27)) hide)
-    )
-    (property "Value" "GND" (at 162.56 13.97 0)
-      (effects (font (size 1.27 1.27)))
-    )
-    (property "Footprint" "" (at 162.56 17.78 0)
-      (effects (font (size 1.27 1.27)) hide)
-    )
-    (property "Datasheet" "" (at 162.56 17.78 0)
-      (effects (font (size 1.27 1.27)) hide)
-    )
-    (pin "1")
-    (instances
-      (project "bc660_breakoutboard"
-        (path "/d627ecd8-d3ea-468a-86f8-a115d49eee0e"
-          (reference "#PWR05") (unit 1)
-        )
-      )
